Commit message: correct a typo in xacro

File: src/my_robot/urdf/my_robot.xacro (robot description, xacro)
@@ -132,5 +132,5 @@
   </link>
 <!-- link for the Lidar  -->
-  <link name='hakuyo'>
+  <link name='hokuyo'>
     <inertial>
       <mass value="1e-5"/>
@@ -151,5 +151,5 @@
       </geometry>
     </visual>
-    <collision name='hakuyo_collision'>
+    <collision name='hokuyo_collision'>
       <origin xyz="0 0 0" rpy="0 0 0"/>
       <geometry>
@@ -184,7 +184,7 @@
   </joint>
 <!--joint for the camera-->
-   <joint type="fixed" name="hakuyo_joint">
+   <joint type="fixed" name="hokuyo_joint">
     <origin xyz="0.15 0.0 0.1" rpy="0 0 0"/>
-    <child link="hakuyo"/>
+    <child link="hokuyo"/>
     <parent link="chassis"/>
     <axis xyz="0 1 0" rpy="0 0 0"/>
